Commit message: Add simple_traj_opt for MultibodyPlant; compiled but have not got a traj soluation yet

File: examples/Goldilocks_models/PlanarWalkerWithTorso.urdf (robot description, URDF)
Before this commit: robot KneedCompassGait, 13 links, 12 joints
Joints:
- joint left_knee_pin: type continuous -> revolute

Commit message: Fix a bug

File: examples/Goldilocks_models/PlanarWalkerWithTorso.urdf (robot description, URDF)
Before this commit: robot KneedCompassGait, 13 links, 12 joints
Joints:
- joint left_knee_pin: limit lower=0 effort=100 -> effort=100
- joint right_knee_pin: limit lower=0 effort=100 -> effort=100
